Commit message: Created robot
Created fncd.xacro file, started adding turtlebot controls

File: urdf/bot.xacro (robot description, xacro)
@@ -1,4 +1,5 @@
 <?xml version='1.0'?>
-<robot name="mogi_bot" xmlns:xacro="http://www.ros.org/wiki/xacro">
+<robot name="fncd_bot" xmlns:xacro="http://www.ros.org/wiki/xacro">
+ <xacro:include filename="$(find fall_and_collision_detection)/urdf/bot.gazebo" />
  <link name="base_footprint"></link>
  <joint name="base_footprint_joint" type="fixed">
@@ -18,8 +19,8 @@
 />
 </inertial>
- <collision name='collision'>
+ <collision name='base_collision'>
 <origin xyz="0 0 0" rpy="0 0 0"/>
 <geometry>
-<box size=".4 .2 .1"/>
+<cylinder radius="0.15" length=".05"/>
 </geometry>
 </collision>
@@ -27,31 +28,81 @@
 <origin xyz="0 0 0" rpy="0 0 0"/>
 <geometry>
-<box size=".4 .2 .1"/>
+<cylinder radius="0.15" length=".05"/>
 </geometry>
 </visual>
- <collision name='rear_caster_collision'>
-<origin xyz="-0.15 0 -0.05" rpy="0 0 0"/>
+ <collision name='caster_collision'>
+<origin xyz="-0.1 0 -0.05" rpy="0 0 0"/>
 <geometry>
-<sphere radius="0.0499"/>
+<sphere radius="0.025"/>
 </geometry>
 </collision>
- <visual name='rear_caster_visual'>
-<origin xyz="-0.15 0 -0.05" rpy="0 0 0"/>
+ <visual name='caster_visual'>
+<origin xyz="-0.1 0 -0.05" rpy="0 0 0"/>
 <geometry>
-<sphere radius="0.05"/>
-</geometry>
-</visual>
- <collision name='front_caster_collision'>
-<origin xyz="0.15 0 -0.05" rpy="0 0 0"/>
-<geometry>
-<sphere radius="0.0499"/>
-</geometry>
-</collision>
- <visual name='front_caster_visual'>
-<origin xyz="0.15 0 -0.05" rpy="0 0 0"/>
-<geometry>
-<sphere radius="0.05"/>
+<sphere radius="0.025"/>
 </geometry>
 </visual>
  </link>
+ <joint type="continuous" name="left_wheel_joint">
+    <origin xyz="0.06 0.1 -0.05" rpy="0 0 0"/>
+    <child link="left_wheel"/>
+    <parent link="base_link"/>
+    <axis xyz="0 1 0" rpy="0 0 0"/>
+    <limit effort="10000" velocity="1000"/>
+    <dynamics damping="1.0" friction="1.0"/>
+  </joint>
+  <link name='left_wheel'>
+    <inertial>
+      <mass value="0.1"/>
+      <origin xyz="0 0 0" rpy="0 1.5707 1.5707"/>
+      <inertia
+          ixx="0.1" ixy="0" ixz="0"
+          iyy="0.1" iyz="0"
+          izz="0.1"
+      />
+    </inertial>
+    <collision name='collision'>
+      <origin xyz="0 0 0" rpy="0 1.5707 1.5707"/>
+      <geometry>
+        <cylinder radius=".025" length=".01"/>
+      </geometry>
+    </collision>
+    <visual name='left_wheel_visual'>
+      <origin xyz="0 0 0" rpy="0 1.5707 1.5707"/>
+      <geometry>
+        <cylinder radius=".025" length=".01"/>
+      </geometry>
+    </visual>
+  </link>
+  <joint type="continuous" name="right_wheel_joint">
+    <origin xyz="0.06 -0.1 -0.05" rpy="0 0 0"/>
+    <child link="right_wheel"/>
+    <parent link="base_link"/>
+    <axis xyz="0 1 0" rpy="0 0 0"/>
+    <limit effort="10000" velocity="1000"/>
+    <dynamics damping="1.0" friction="1.0"/>
+  </joint>
+  <link name='right_wheel'>
+    <inertial>
+      <mass value="5.0"/>
+      <origin xyz="0 0 0" rpy="0 1.5707 1.5707"/>
+      <inertia
+          ixx="0.1" ixy="0" ixz="0"
+          iyy="0.1" iyz="0"
+          izz="0.1"
+      />
+    </inertial>
+    <collision name='collision'>
+      <origin xyz="0 0 0" rpy="0 1.5707 1.5707"/>
+      <geometry>
+        <cylinder radius=".025" length=".01"/>
+      </geometry>
+    </collision>
+    <visual name='right_wheel_visual'>
+      <origin xyz="0 0 0" rpy="0 1.5707 1.5707"/>
+      <geometry>
+        <cylinder radius=".025" length=".01"/>
+      </geometry>
+    </visual>
+  </link>
 </robot>

Commit message: Lidar added

File: urdf/bot.xacro (robot description, xacro)
@@ -106,3 +106,33 @@
     </visual>
   </link>
+  <!-- Lidar -->
+  <joint type="fixed" name="scan_joint">
+    <origin xyz="0.0 0 0.05" rpy="0 0 0"/>
+    <child link="scan_link"/>
+    <parent link="base_link"/>
+    <axis xyz="0 1 0" rpy="0 0 0"/>
+  </joint>
+  <link name='scan_link'>
+    <inertial>
+      <mass value="1e-5"/>
+      <origin xyz="0 0 0" rpy="0 0 0"/>
+      <inertia
+          ixx="1e-6" ixy="0" ixz="0"
+          iyy="1e-6" iyz="0"
+          izz="1e-6"
+      />
+    </inertial>
+    <collision name='collision'>
+      <origin xyz="0 0 0" rpy="0 0 0"/>
+      <geometry>
+        <box size=".1 .1 .1"/>
+      </geometry>
+    </collision>
+    <visual name='scan_link_visual'>
+      <origin xyz="0 0 0" rpy="0 0 0"/>
+      <geometry>
+        <mesh filename = "package://bme_gazebo_sensors/meshes/lidar.dae"/>
+      </geometry>
+    </visual>
+  </link>
 </robot>

Commit message: IR sensors added

File: urdf/bot.xacro (robot description, xacro)
@@ -8,5 +8,5 @@
 <child link="base_link" />
 </joint>
- <link name='base_link'>
+<link name='base_link'>
 <pose>0 0 0.1 0 0 0</pose>
  <inertial>
@@ -136,3 +136,84 @@
     </visual>
   </link>
+  <!-- IR sensor 1 -->
+  <joint type="fixed" name="ir_front_joint">
+    <origin xyz="0.14 0 -0.030" rpy="0 1.56 0"/>
+    <child link="base_ir_front"/>
+    <parent link="base_link"/>
+    <axis xyz="1 0 0" rpy="0 0 0"/>
+  </joint>
+  <link name="base_ir_front">
+    <collision>
+      <origin xyz="0 0 0" rpy="0 0 0"/>
+      <geometry>
+        <box size="0.01 0.01 0.01"/>
+      </geometry>
+    </collision>
+    <visual>
+      <origin xyz="0 0 0" rpy="0 0 0"/>
+      <geometry>
+        <box size="0.01 0.01 0.01"/>
+      </geometry>
+      <material name="green"/>
+    </visual>
+    <inertial>
+      <mass value="1e-5" />
+      <origin xyz="0 0 0" rpy="0 0 0"/>
+      <inertia ixx="1e-6" ixy="0" ixz="0" iyy="1e-6" iyz="0"      izz="1e-6" />
+    </inertial>
+  </link>
+  <!-- IR sensor 2 -->
+  <joint type="fixed" name="ir_left_joint">
+    <origin xyz="0.0 -0.14 -0.030" rpy="0 1.56 0"/>
+    <child link="base_ir_left"/>
+    <parent link="base_link"/>
+    <axis xyz="1 0 0" rpy="0 0 0"/>
+  </joint>
+  <link name="base_ir_left">
+    <collision>
+      <origin xyz="0 0 0" rpy="0 0 0"/>
+      <geometry>
+        <box size="0.01 0.01 0.01"/>
+      </geometry>
+    </collision>
+    <visual>
+      <origin xyz="0 0 0" rpy="0 0 0"/>
+      <geometry>
+        <box size="0.01 0.01 0.01"/>
+      </geometry>
+      <material name="green"/>
+    </visual>
+    <inertial>
+      <mass value="1e-5" />
+      <origin xyz="0 0 0" rpy="0 0 0"/>
+      <inertia ixx="1e-6" ixy="0" ixz="0" iyy="1e-6" iyz="0"      izz="1e-6" />
+    </inertial>
+  </link>
+    <!-- IR sensor 3 -->
+  <joint type="fixed" name="ir_right_joint">
+    <origin xyz="0.0 0.14 -0.030" rpy="0 1.56 0"/>
+    <child link="base_ir_right"/>
+    <parent link="base_link"/>
+    <axis xyz="1 0 0" rpy="0 0 0"/>
+  </joint>
+  <link name="base_ir_right">
+    <collision>
+      <origin xyz="0 0 0" rpy="0 0 0"/>
+      <geometry>
+        <box size="0.01 0.01 0.01"/>
+      </geometry>
+    </collision>
+    <visual>
+      <origin xyz="0 0 0" rpy="0 0 0"/>
+      <geometry>
+        <box size="0.01 0.01 0.01"/>
+      </geometry>
+      <material name="green"/>
+    </visual>
+    <inertial>
+      <mass value="1e-5" />
+      <origin xyz="0 0 0" rpy="0 0 0"/>
+      <inertia ixx="1e-6" ixy="0" ixz="0" iyy="1e-6" iyz="0"      izz="1e-6" />
+    </inertial>
+  </link>
 </robot>

Commit message: Modified bot.xacro
Robot can now turn in place, has two casters

File: urdf/bot.xacro (robot description, xacro)
@@ -20,5 +20,5 @@
 </inertial>
  <collision name='base_collision'>
-<origin xyz="0 0 0" rpy="0 0 0"/>
+<origin xyz="0 0 -0.025" rpy="0 0 0"/>
 <geometry>
 <cylinder radius="0.15" length=".05"/>
@@ -26,5 +26,5 @@
 </collision>
  <visual name='base_link_visual'>
-<origin xyz="0 0 0" rpy="0 0 0"/>
+<origin xyz="0 0 -0.025" rpy="0 0 0"/>
 <geometry>
 <cylinder radius="0.15" length=".05"/>
@@ -34,5 +34,5 @@
 <origin xyz="-0.1 0 -0.05" rpy="0 0 0"/>
 <geometry>
-<sphere radius="0.025"/>
+<sphere radius="0.02"/>
 </geometry>
 </collision>
@@ -40,10 +40,34 @@
 <origin xyz="-0.1 0 -0.05" rpy="0 0 0"/>
 <geometry>
-<sphere radius="0.025"/>
+<sphere radius="0.02"/>
 </geometry>
 </visual>
+<collision name='caster2_collision'>
+  <origin xyz="0.1 0 -0.05" rpy="0 0 0"/>
+  <geometry>
+  <sphere radius="0.02"/>
+  </geometry>
+  </collision>
+   <visual name='caster2_visual'>
+  <origin xyz="0.1 0 -0.05" rpy="0 0 0"/>
+  <geometry>
+  <sphere radius="0.02"/>
+  </geometry>
+  </visual>
+  <collision name='indicator_collision'>
+    <origin xyz="0.1 0 0.001" rpy="0 0 0"/>
+    <geometry>
+    <sphere radius="0.01"/>
+    </geometry>
+    </collision>
+     <visual name='indicator_visual'>
+    <origin xyz="0.1 0 0.001" rpy="0 0 0"/>
+    <geometry>
+    <sphere radius="0.01"/>
+    </geometry>
+    </visual>
  </link>
  <joint type="continuous" name="left_wheel_joint">
-    <origin xyz="0.06 0.1 -0.05" rpy="0 0 0"/>
+    <origin xyz="0.00 0.1 -0.05" rpy="0 0 0"/>
     <child link="left_wheel"/>
     <parent link="base_link"/>
@@ -76,5 +100,5 @@
   </link>
   <joint type="continuous" name="right_wheel_joint">
-    <origin xyz="0.06 -0.1 -0.05" rpy="0 0 0"/>
+    <origin xyz="0.00 -0.1 -0.05" rpy="0 0 0"/>
     <child link="right_wheel"/>
     <parent link="base_link"/>

Commit message: removed <material name=green> lines from gazeboo file
exit

File: urdf/bot.xacro (robot description, xacro)
@@ -179,5 +179,4 @@
         <box size="0.01 0.01 0.01"/>
       </geometry>
-      <material name="green"/>
     </visual>
     <inertial>
@@ -206,5 +205,4 @@
         <box size="0.01 0.01 0.01"/>
       </geometry>
-      <material name="green"/>
     </visual>
     <inertial>
@@ -233,5 +231,4 @@
         <box size="0.01 0.01 0.01"/>
       </geometry>
-      <material name="green"/>
     </visual>
     <inertial>

Commit message: gmapping setup

File: urdf/bot.xacro (robot description, xacro)
@@ -163,5 +163,5 @@
   <!-- IR sensor 1 -->
   <joint type="fixed" name="ir_front_joint">
-    <origin xyz="0.14 0 -0.030" rpy="0 1.56 0"/>
+    <origin xyz="0.14 0 -0.05" rpy="0 1.56 0"/>
     <child link="base_ir_front"/>
     <parent link="base_link"/>
@@ -189,5 +189,5 @@
   <!-- IR sensor 2 -->
   <joint type="fixed" name="ir_left_joint">
-    <origin xyz="0.0 -0.14 -0.030" rpy="0 1.56 0"/>
+    <origin xyz="0.0 -0.14 -0.05" rpy="0 1.56 0"/>
     <child link="base_ir_left"/>
     <parent link="base_link"/>
@@ -215,5 +215,5 @@
     <!-- IR sensor 3 -->
   <joint type="fixed" name="ir_right_joint">
-    <origin xyz="0.0 0.14 -0.030" rpy="0 1.56 0"/>
+    <origin xyz="0.0 0.14 -0.05" rpy="0 1.56 0"/>
     <child link="base_ir_right"/>
     <parent link="base_link"/>

Commit message: mapping fix

File: urdf/bot.xacro (robot description, xacro)
@@ -34,5 +34,5 @@
 <origin xyz="-0.1 0 -0.05" rpy="0 0 0"/>
 <geometry>
-<sphere radius="0.02"/>
+<sphere radius="0.0245"/>
 </geometry>
 </collision>
@@ -40,5 +40,5 @@
 <origin xyz="-0.1 0 -0.05" rpy="0 0 0"/>
 <geometry>
-<sphere radius="0.02"/>
+<sphere radius="0.0245"/>
 </geometry>
 </visual>
@@ -46,5 +46,5 @@
   <origin xyz="0.1 0 -0.05" rpy="0 0 0"/>
   <geometry>
-  <sphere radius="0.02"/>
+  <sphere radius="0.0245"/>
   </geometry>
   </collision>
@@ -52,5 +52,5 @@
   <origin xyz="0.1 0 -0.05" rpy="0 0 0"/>
   <geometry>
-  <sphere radius="0.02"/>
+  <sphere radius="0.0245"/>
   </geometry>
   </visual>

Commit message: random_move script fix

File: urdf/bot.xacro (robot description, xacro)
@@ -69,5 +69,5 @@
  </link>
  <joint type="continuous" name="left_wheel_joint">
-    <origin xyz="0.00 0.1 -0.05" rpy="0 0 0"/>
+    <origin xyz="0.00 0.08 -0.05" rpy="0 0 0"/>
     <child link="left_wheel"/>
     <parent link="base_link"/>
@@ -100,5 +100,5 @@
   </link>
   <joint type="continuous" name="right_wheel_joint">
-    <origin xyz="0.00 -0.1 -0.05" rpy="0 0 0"/>
+    <origin xyz="0.00 -0.08 -0.05" rpy="0 0 0"/>
     <child link="right_wheel"/>
     <parent link="base_link"/>
@@ -132,5 +132,5 @@
   <!-- Lidar -->
   <joint type="fixed" name="scan_joint">
-    <origin xyz="0.0 0 0.05" rpy="0 0 0"/>
+    <origin xyz="0.0 0 0.03" rpy="0 0 0"/>
     <child link="scan_link"/>
     <parent link="base_link"/>

Commit message: Range mapping and map merging

File: urdf/bot.xacro (robot description, xacro)
@@ -19,5 +19,5 @@
 />
 </inertial>
- <collision name='base_collision'>
+<collision name='base_collision'>
 <origin xyz="0 0 -0.025" rpy="0 0 0"/>
 <geometry>

Commit message: Deleted unnecessary files, fixed dimensions, added meshes to <visual> of xacro file

File: urdf/bot.xacro (robot description, xacro)
@@ -29,4 +29,5 @@
 <geometry>
 <cylinder radius="0.15" length=".05"/>
+<mesh filename = "package://fall_and_collision_detection/meshes/bot_base.dae"/>
 </geometry>
 </visual>
@@ -41,4 +42,5 @@
 <geometry>
 <sphere radius="0.0245"/>
+<mesh filename = "package://fall_and_collision_detection/meshes/caster.dae"/>
 </geometry>
 </visual>
@@ -53,4 +55,5 @@
   <geometry>
   <sphere radius="0.0245"/>
+  <mesh filename = "package://fall_and_collision_detection/meshes/caster.dae"/>
   </geometry>
   </visual>
@@ -96,4 +99,5 @@
       <geometry>
         <cylinder radius=".025" length=".01"/>
+        <mesh filename = "package://fall_and_collision_detection/meshes/wheel.dae"/>
       </geometry>
     </visual>
@@ -127,4 +131,5 @@
       <geometry>
         <cylinder radius=".025" length=".01"/>
+        <mesh filename = "package://fall_and_collision_detection/meshes/wheel.dae"/>
       </geometry>
     </visual>

Commit message: Readme and some fixes

File: urdf/bot.xacro (robot description, xacro)
@@ -3,59 +3,59 @@
  <xacro:include filename="$(find fall_and_collision_detection)/urdf/bot.gazebo" />
  <link name="base_footprint"></link>
- <joint name="base_footprint_joint" type="fixed">
-<origin xyz="0 0 0" rpy="0 0 0" />
-<parent link="base_footprint"/>
-<child link="base_link" />
+<joint name="base_footprint_joint" type="fixed">
+  <origin xyz="0 0 0" rpy="0 0 0" />
+  <parent link="base_footprint"/>
+  <child link="base_link" />
 </joint>
 <link name='base_link'>
 <pose>0 0 0.1 0 0 0</pose>
- <inertial>
-<mass value="15.0"/>
-<origin xyz="0 0 0" rpy="0 0 0"/>
-<inertia
-ixx="0.1" ixy="0" ixz="0"
-iyy="0.1" iyz="0"
-izz="0.1"
-/>
+<inertial>
+  <mass value="15.0"/>
+  <origin xyz="0 0 0" rpy="0 0 0"/>
+  <inertia
+    ixx="0.1" ixy="0" ixz="0"
+    iyy="0.1" iyz="0"
+    izz="0.1"
+  />
 </inertial>
 <collision name='base_collision'>
-<origin xyz="0 0 -0.025" rpy="0 0 0"/>
-<geometry>
-<cylinder radius="0.15" length=".05"/>
-</geometry>
+  <origin xyz="0 0 -0.025" rpy="0 0 0"/>
+  <geometry>
+    <cylinder radius="0.15" length=".05"/>
+  </geometry>
 </collision>
- <visual name='base_link_visual'>
-<origin xyz="0 0 -0.025" rpy="0 0 0"/>
-<geometry>
-<cylinder radius="0.15" length=".05"/>
-<mesh filename = "package://fall_and_collision_detection/meshes/bot_base.dae"/>
-</geometry>
+<visual name='base_link_visual'>
+  <origin xyz="0 0 -0.025" rpy="0 0 0"/>
+  <geometry>
+    <!-- <cylinder radius="0.15" length=".05"/> -->
+    <mesh filename = "package://fall_and_collision_detection/meshes/bot_base.dae"/>
+  </geometry>
 </visual>
- <collision name='caster_collision'>
-<origin xyz="-0.1 0 -0.05" rpy="0 0 0"/>
-<geometry>
-<sphere radius="0.0245"/>
-</geometry>
+<collision name='caster_collision'>
+  <origin xyz="-0.1 0 -0.05" rpy="0 0 0"/>
+  <geometry>
+    <sphere radius="0.0245"/>
+  </geometry>
 </collision>
- <visual name='caster_visual'>
-<origin xyz="-0.1 0 -0.05" rpy="0 0 0"/>
-<geometry>
-<sphere radius="0.0245"/>
-<mesh filename = "package://fall_and_collision_detection/meshes/caster.dae"/>
-</geometry>
+<visual name='caster_visual'>
+  <origin xyz="-0.1 0 -0.05" rpy="0 0 0"/>
+  <geometry>
+    <!-- <sphere radius="0.0245"/> -->
+    <mesh filename = "package://fall_and_collision_detection/meshes/caster.dae"/>
+  </geometry>
 </visual>
 <collision name='caster2_collision'>
   <origin xyz="0.1 0 -0.05" rpy="0 0 0"/>
   <geometry>
-  <sphere radius="0.0245"/>
-  </geometry>
-  </collision>
-   <visual name='caster2_visual'>
+    <sphere radius="0.0245"/>
+  </geometry>
+</collision>
+<visual name='caster2_visual'>
   <origin xyz="0.1 0 -0.05" rpy="0 0 0"/>
   <geometry>
-  <sphere radius="0.0245"/>
-  <mesh filename = "package://fall_and_collision_detection/meshes/caster.dae"/>
-  </geometry>
-  </visual>
+    <!-- <sphere radius="0.0245"/> -->
+    <mesh filename = "package://fall_and_collision_detection/meshes/caster.dae"/>
+  </geometry>
+</visual>
   <collision name='indicator_collision'>
     <origin xyz="0.1 0 0.001" rpy="0 0 0"/>
@@ -98,5 +98,5 @@
       <origin xyz="0 0 0" rpy="0 1.5707 1.5707"/>
       <geometry>
-        <cylinder radius=".025" length=".01"/>
+        <!-- <cylinder radius=".025" length=".01"/> -->
         <mesh filename = "package://fall_and_collision_detection/meshes/wheel.dae"/>
       </geometry>
@@ -130,5 +130,5 @@
       <origin xyz="0 0 0" rpy="0 1.5707 1.5707"/>
       <geometry>
-        <cylinder radius=".025" length=".01"/>
+        <!-- <cylinder radius=".025" length=".01"/> -->
         <mesh filename = "package://fall_and_collision_detection/meshes/wheel.dae"/>
       </geometry>

Commit message: Fix

File: urdf/bot.xacro (robot description, xacro)
@@ -161,6 +161,5 @@
       <origin xyz="0 0 0" rpy="0 0 0"/>
       <geometry>
-        <!--  TODO : use own mesh instead-->
-        <mesh filename = "package://bme_gazebo_sensors/meshes/lidar.dae"/>
+        <mesh filename = "package://fall_and_collision_detection/meshes/lidar.dae"/>
       </geometry>
     </visual>
